Commit message: edit point error

File: urdf/gimbal_v2.urdf (robot description, URDF)
Before this commit: robot gimbal_v2, 7 links, 6 joints
Joints:
- joint pitch_joint: origin xyz=0 0.094 0.136 rpy=0 0 0 -> xyz=0 0.094 0.136 rpy=0 0 -0.085
- joint roll_joint: origin xyz=0 -0.094 0 rpy=0 0 0 -> xyz=0 -0.094 0 rpy=-2 0 0
- joint yaw_joint: origin xyz=0 0 0 rpy=0 0 0 -> xyz=0 0 0 rpy=0 0 -1.31
